File: PCB/TPI_v1.kicad_sch (KiCad schematic)
At the start: 7 parts, among them J1 Raspberry pi zero w, J2 BME280, J3 BME280, J4 MQ135, U1 BMI160, U2 DS18B20

Commit message: PCB update
Parts:
- removed J3: BME280, Connector_JST:JST_PH_S4B-PH-K_1x04_P2.00mm_Horizontal, symbol Connector_Generic:Conn_01x04
- added C1: 100n, Capacitor_THT:C_Disc_D3.0mm_W1.6mm_P2.50mm, symbol Device:C
- added D1: LED, symbol Device:LED
- added J3: SIG2991, Connector_JST:JST_XH_S2B-XH-A-1_1x02_P2.50mm_Horizontal, symbol Connector_Generic:Conn_01x02
- added J5: Buck, Connector_PinSocket_2.54mm:PinSocket_2x01_P2.54mm_Vertical, symbol Connector_Generic:Conn_01x02
- added R2: 10k, Resistor_THT:R_Axial_DIN0207_L6.3mm_D2.5mm_P7.62mm_Horizontal, symbol Device:R
- added R3: 1K, Resistor_THT:R_Axial_DIN0207_L6.3mm_D2.5mm_P7.62mm_Horizontal, symbol Device:R
- added U3: MCP3008, Package_DIP:DIP-16_W7.62mm, symbol Analog_ADC:MCP3008
- added U4: DS18B20_2, Connector_JST:JST_XH_S3B-XH-A-1_1x03_P2.50mm_Horizontal, symbol Sensor_Temperature:DS18B20
- added U5: DS18B20_3, Connector_JST:JST_XH_S3B-XH-A-1_1x03_P2.50mm_Horizontal, symbol Sensor_Temperature:DS18B20
- added U6: DS18B20_4, Connector_JST:JST_XH_S3B-XH-A-1_1x03_P2.50mm_Horizontal, symbol Sensor_Temperature:DS18B20
- J2: footprint Connector_JST:JST_PH_S4B-PH-K_1x04_P2.00mm_Horizontal -> Connector_JST:JST_XH_S4B-XH-A-1_1x04_P2.50mm_Horizontal
- J4: footprint (none) -> Connector_JST:JST_XH_B3B-XH-A_1x03_P2.50mm_Vertical
- U2: value DS18B20 -> DS18B20_1; footprint Connector_JST:JST_PH_S3B-PH-K_1x03_P2.00mm_Horizontal -> Connector_JST:JST_XH_S3B-XH-A-1_1x03_P2.50mm_Horizontal
Connections:
- net +3.3V: no longer U1.1 (VIN)
- net +5V: now also J1.4 (5V), U1.1 (VIN), J5.1 (Pin_1), R2.1, R3.1, U3.15 (Vref), U3.16 (Vdd), U4.3 (V_{DD}), U5.3 (V_{DD}), U6.3 (V_{DD})
- net DQ: now also U4.2 (DQ), U5.2 (DQ), U6.2 (DQ)
- net GND: now also C1.2, D1.1 (K), J3.2 (Pin_2), J5.2 (Pin_2), U3.14 (AGND), U3.9 (DGND), U4.1 (GND), U5.1 (GND), U6.1 (GND); no longer J1.20 (GND)
- net ADC0: now reaches J4.2 (Pin_2)
- net ADC0: now also U3.1 (CH0)
- net MOSI: now reaches J1.19 (GPIO10)
- net MOSI: now also U3.11 (Din)
- net MISO: now reaches J1.21 (GPIO9)
- net MISO: now also U3.12 (Dout)
- net SCLK: now reaches J1.23 (GPIO11)
- net SCLK: now also U3.13 (CLK)
- net ~{CS}: now reaches J1.24 (GPIO8)
- net ~{CS}: now also U3.10 (~{CS}/SHDN)
- new net: D1.2 (A), R3.2
- new net ADC1: C1.1, J3.1 (Pin_1), R2.2, U3.2 (CH1)
- no-connect marks 11 -> 36
Other:
- note added: "Conversor ADC (MCP3008-I/P)"
- note added: "Iluminacion"
- note added: "Sensor de Humedad (SIG2991)"
- note added: "Sensores Analogicos"
- title: (none) -> WALL-E Hat
- moved on the sheet: J1, J2, J4, R1, U1, U2

Commit message: PCB
Se cambio el voltaje del sensor BME280
Connections:
- net +3.3V: now also J2.3 (Pin_3)
- net +5V: no longer J2.3 (Pin_3)
Changed lines of the file:
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@@
 	(wire
 		(pts
+			(xy 64.77 81.915) (xy 64.77 83.185)
+		)
+		(stroke
+			(width 0)
+			(type default)
+		)
+	)
+	(wire
+		(pts
 			(xy 105.41 71.755) (xy 107.95 71.755)
 		)
@@
 	)
 	(symbol
+		(lib_id "power:+3.3V")
+		(at 64.77 81.915 0)
+		(unit 1)
+		(exclude_from_sim no)
+		(in_bom yes)
+		(on_board yes)
+		(dnp no)
+		(fields_autoplaced yes)
+		(property "Reference" "#PWR06"
+			(at 64.77 85.725 0)
+			(effects
+				(font
+					(size 1.27 1.27)
+				)
+				(hide yes)
+			)
+		)
+		(property "Value" "+3.3V"
+			(at 64.77 77.47 0)
+			(effects
+				(font
+					(size 1.27 1.27)
+				)
+			)
+		)
+		(property "Footprint" ""
+			(at 64.77 81.915 0)
+			(effects
+				(font
+					(size 1.27 1.27)
+				)
+				(hide yes)
+			)
+		)
+		(property "Datasheet" ""
+			(at 64.77 81.915 0)
+			(effects
+				(font
+					(size 1.27 1.27)
+				)
+				(hide yes)
+			)
+		)
+		(property "Description" "Power symbol creates a global label with name \"+3.3V\""
+			(at 64.77 81.915 0)
+			(effects
+				(font
+					(size 1.27 1.27)
+				)
+				(hide yes)
+			)
+		)
+		(pin "1"
+		)
+		(instances
+			(project ""
+				(path "/79131faf-b6e1-4903-a0d0-df18876f9f0e"
+					(reference "#PWR06")
+					(unit 1)
+				)
+			)
+		)
+	)
+	(symbol
 		(lib_id "power:GND")
 		(at 240.03 74.93 0)
@@
 					(unit 1)
 				)
-			)
-		)
-	)
-	(symbol
-		(lib_id "power:+5V")
-		(at 64.77 83.185 0)
-		(unit 1)
-		(exclude_from_sim no)
-		(in_bom yes)
-		(on_board yes)
-		(dnp no)
-		(property "Reference" "#PWR06"
-			(at 64.77 86.995 0)
-			(effects
-				(font
-					(size 1.27 1.27)
-				)
-				(hide yes)
-			)
-		)
-		(property "Value" "+5V"
-			(at 67.056 81.915 90)
-			(effects
-				(font
-					(size 1.27 1.27)
-				)
-			)
-		)
-		(property "Footprint" ""
-			(at 64.77 83.185 0)
-			(effects
-				(font
-					(size 1.27 1.27)
-				)
-				(hide yes)
-			)
-		)
-		(property "Datasheet" ""
-			(at 64.77 83.185 0)
-			(effects
-				(font
-					(size 1.27 1.27)
-				)
-				(hide yes)
-			)
-		)
-		(property "Description" "Power symbol creates a global label with name \"+5V\""
-			(at 64.77 83.185 0)
-			(effects
-				(font
-					(size 1.27 1.27)
-				)
-				(hide yes)
-			)
-		)
-		(pin "1"
-		)
-		(instances
-			(project ""
-				(path "/79131faf-b6e1-4903-a0d0-df18876f9f0e"
-					(reference "#PWR06")
-					(unit 1)
-				)

Commit message: PCB update
V2 PCB
Parts:
- J2: footprint Connector_JST:JST_XH_S4B-XH-A-1_1x04_P2.50mm_Horizontal -> Connector_JST:JST_XH_B4B-XH-A_1x04_P2.50mm_Vertical
- J4: footprint Connector_JST:JST_XH_B3B-XH-A_1x03_P2.50mm_Vertical -> Connector_JST:JST_XH_S3B-XH-A-1_1x03_P2.50mm_Horizontal
- U2: value DS18B20_1 -> DS18B20_2
- U5: value DS18B20_3 -> DS18B20_2; footprint Connector_JST:JST_XH_S3B-XH-A-1_1x03_P2.50mm_Horizontal -> Connector_JST:JST_XH_B3B-XH-A_1x03_P2.50mm_Vertical
- U6: value DS18B20_4 -> DS18B20_2; footprint Connector_JST:JST_XH_S3B-XH-A-1_1x03_P2.50mm_Horizontal -> Connector_JST:JST_XH_B3B-XH-A_1x03_P2.50mm_Vertical
Connections:
- net +3.3V: now also J1.17 (3.3V), U1.1 (VIN)
- net +5V: now also J4.3 (Pin_1); no longer J4.1 (Pin_1), U1.1 (VIN)
- net ADC0: now also J4.1 (Pin_2); no longer J4.2 (Pin_2)
- net DQ: now also U2.1 (DQ), U4.1 (DQ), U5.1 (DQ), U6.1 (DQ); no longer U2.2 (DQ), U4.2 (DQ), U5.2 (DQ), U6.2 (DQ)
- net GND: now also J4.2 (Pin_3), U2.2 (GND), U4.2 (GND), U5.2 (GND), U6.2 (GND); no longer J4.3 (Pin_3), U2.1 (GND), U4.1 (GND), U5.1 (GND), U6.1 (GND)
- net ~{CS}: now also J1.15 (GPIO22); no longer J1.24 (GPIO8)
- no-connect marks 36 -> 34

Commit message: General update
Parts:
- added D2: LED, LED_THT:LED_D3.0mm, symbol Device:LED
- added R4: 2.2K, Resistor_THT:R_Axial_DIN0207_L6.3mm_D2.5mm_P7.62mm_Horizontal, symbol Device:R
- D1: footprint (none) -> LED_THT:LED_D3.0mm
- R3: value 1K -> 2.2K
Connections:
- net GND: now also D2.1 (K)
- net Server: now reaches J1.37 (GPIO26)
- net Server: now also R4.1
- new net: D2.2 (A), R4.2
- no-connect marks 34 -> 33
Other:
- moved on the sheet: D1, R3
